File: tux_badge.kicad_sch (KiCad schematic)
At the start: 4 parts, among them SW1 SW_Push

Commit message: first order
Parts:
- BT1: LCSC (none) -> C964829
- D1: value LED -> Yellow; LCSC (none) -> C434436
- R1: value R -> 62; LCSC (none) -> C865596
- SW1: LCSC (none) -> C202424
Changed lines of the file:
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@@
       (effects (font (size 1.27 1.27)) (justify right))
     )
-    (property "Value" "LED" (id 1) (at 162.56 106.9974 90)
+    (property "Value" "Yellow" (id 1) (at 162.56 106.9974 90)
       (effects (font (size 1.27 1.27)) (justify right))
     )
@@
     )
     (property "Datasheet" "~" (id 3) (at 158.75 104.14 0)
+      (effects (font (size 1.27 1.27)) hide)
+    )
+    (property "LCSC" "C434436" (id 4) (at 158.75 104.14 90)
       (effects (font (size 1.27 1.27)) hide)
     )
@@
     )
     (property "Value" "SW_Push" (id 1) (at 162.433 77.4699 90)
-      (effects (font (size 1.27 1.27)) (justify left))
+      (effects (font (size 1.27 1.27)) (justify left) hide)
     )
     (property "Footprint" "Button_Switch_SMD:SW_SPST_SKQG_WithStem" (id 2) (at 163.83 76.2 0)
@@
     )
     (property "Datasheet" "~" (id 3) (at 163.83 76.2 0)
+      (effects (font (size 1.27 1.27)) hide)
+    )
+    (property "LCSC" "C202424" (id 4) (at 158.75 76.2 90)
       (effects (font (size 1.27 1.27)) hide)
     )
@@
       (effects (font (size 1.27 1.27)) (justify left))
     )
-    (property "Value" "R" (id 1) (at 161.29 91.4399 0)
+    (property "Value" "62" (id 1) (at 161.29 91.4399 0)
       (effects (font (size 1.27 1.27)) (justify left))
     )
@@
     )
     (property "Datasheet" "~" (id 3) (at 158.75 90.17 0)
+      (effects (font (size 1.27 1.27)) hide)
+    )
+    (property "LCSC" "C865596" (id 4) (at 158.75 90.17 0)
       (effects (font (size 1.27 1.27)) hide)
     )
@@
     )
     (property "Datasheet" "~" (id 3) (at 125.73 88.646 90)
+      (effects (font (size 1.27 1.27)) hide)
+    )
+    (property "LCSC" "C964829" (id 4) (at 125.73 90.17 0)
       (effects (font (size 1.27 1.27)) hide)
     )
@@
     )
     (path "/11471a6b-4e22-40fa-82e7-fea3729faabb"
-      (reference "D1") (unit 1) (value "LED") (footprint "LED_SMD:LED_0805_2012Metric_Pad1.15x1.40mm_HandSolder")
+      (reference "D1") (unit 1) (value "Yellow") (footprint "LED_SMD:LED_0805_2012Metric_Pad1.15x1.40mm_HandSolder")
     )
     (path "/b9ffe1be-0254-4cff-b06a-d8c99588d721"
-      (reference "R1") (unit 1) (value "R") (footprint "Resistor_SMD:R_0805_2012Metric_Pad1.20x1.40mm_HandSolder")
+      (reference "R1") (unit 1) (value "62") (footprint "Resistor_SMD:R_0805_2012Metric_Pad1.20x1.40mm_HandSolder")
     )
     (path "/32b55113-c42d-4fbc-8c9a-5c07a30e5682"

Commit message: adding BOM and fixing losed silkscreen icons
Other:
- title: (none) -> Tux-Badge
Changed lines of the file:
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@@
 (kicad_sch (version 20211123) (generator eeschema)
   (paper "A4")
+  (title_block
+    (title "Tux-Badge")
+    (date "2023-07-01")
+    (rev "1.0")
+  )
   (junction (at 142.24 67.31) (diameter 0) (color 0 0 0 0)
   )
